Commit message: added target velocities; no help

File: urdf/TwoJointRobot.urdf (robot description, URDF)
Before this commit: robot TwoJointRobot, 4 links, 3 joints
Joints:
- joint joint_1: limit lower=-3.14 upper=3.14 effort=10000 velocity=5 -> lower=-3.14 upper=3.14 effort=1000000 velocity=50000
- joint joint_2: limit lower=-3.14 upper=3.14 effort=10000 velocity=5 -> lower=-3.14 upper=3.14 effort=1000000 velocity=50000
