Commit message: xacro urdf works!

File: urdf/sdab.xacro (robot description, xacro)
@@ -51,5 +51,5 @@
 			<parent link="body"/>
 			<child link="${prefix}wing_spar"/>
-			<axis xyz="0 0 -${sign}"/>
+			<axis xyz="0 0 ${-1 * sign}"/>
 			<origin xyz="0.0 0 0.1" rpy="0 0 0"/>
 		</joint>
@@ -57,5 +57,5 @@
 			<parent link="${prefix}wing_spar"/>
 			<child link="${prefix}wing_membrane"/>
-			<axis xyz="0 -${sign} 0"/>
+			<axis xyz="0 ${-1 * sign} 0"/>
 			<origin xyz="0.0 0 0.0" rpy="0 0 0"/>
 		</joint>

Commit message: parameters modularized to top of file

File: urdf/sdab.xacro (robot description, xacro)
@@ -7,4 +7,16 @@
 	<!-- Define parameters -->
 	<xacro:property name="pi" value="3.14159265359"/>
+	<xacro:property name="wbody" value="0.05"/>
+	<xacro:property name="lbody" value="0.2"/>
+	<!-- radial distance from center to start of wing -->
+	<xacro:property name="RwingOffset" value="0.04"/>
+	<!-- diameter of spar -->
+	<xacro:property name="dspar" value="0.01"/>
+	<!-- radial wing length -->
+	<xacro:property name="Rwing" value="0.12"/>
+	<!-- mean chord length -->
+	<xacro:property name="cbar" value="0.06"/>
+	<!-- vertical offset of wing attachment point from COM -->
+	<xacro:property name="d" value="0.1"/>
 	<!-- Define materials -->
 	<material name="Black1">
@@ -22,5 +34,5 @@
 			<origin xyz="0 0 0.0" rpy="0 0 0"/>
 			<geometry>
-				<box size="0.05 0.05 0.2"/>
+				<box size="${wbody} ${wbody} ${lbody}"/>
 			</geometry>
 	    <material name="Blue1"/>
@@ -31,7 +43,7 @@
 		<link name="${prefix}wing_spar">
 			<visual>
-				<origin xyz="0 ${sign * 0.08} 0.0" rpy="0 0 0"/>
+				<origin xyz="0 ${sign * 0.5 * (Rwing + RwingOffset)} 0.0" rpy="0 0 0"/>
 				<geometry>
-					<box size="0.01 0.16 0.01"/>
+					<box size="${dspar} ${RwingOffset + Rwing} ${dspar}"/>
 				</geometry>
 				<material name="Black1"/>
@@ -40,7 +52,7 @@
 		<link name="${prefix}wing_membrane">
 			<visual>
-				<origin xyz="0 ${sign * 0.08} -0.03" rpy="0 0 0"/>
+				<origin xyz="0 ${sign * 0.5 * (Rwing + RwingOffset)} ${-0.5 * cbar}" rpy="0 0 0"/>
 				<geometry>
-					<box size="0.01 0.12 0.06"/>
+					<box size="${dspar} ${Rwing} ${cbar}"/>
 				</geometry>
 				<material name="Gray1"/>
@@ -52,5 +64,5 @@
 			<child link="${prefix}wing_spar"/>
 			<axis xyz="0 0 ${-1 * sign}"/>
-			<origin xyz="0.0 0 0.1" rpy="0 0 0"/>
+			<origin xyz="0.0 0 ${d}" rpy="0 0 0"/>
 		</joint>
 		<joint name="${prefix}wing_hinge" type="continuous">

Commit message: scale shrunk to actual

File: urdf/sdab.xacro (robot description, xacro)
@@ -7,16 +7,16 @@
 	<!-- Define parameters -->
 	<xacro:property name="pi" value="3.14159265359"/>
-	<xacro:property name="wbody" value="0.05"/>
-	<xacro:property name="lbody" value="0.2"/>
+	<xacro:property name="wbody" value="0.003"/>
+	<xacro:property name="lbody" value="0.012"/>
 	<!-- radial distance from center to start of wing -->
-	<xacro:property name="RwingOffset" value="0.04"/>
+	<xacro:property name="RwingOffset" value="0.004"/>
 	<!-- diameter of spar -->
-	<xacro:property name="dspar" value="0.01"/>
+	<xacro:property name="dspar" value="0.001"/>
 	<!-- radial wing length -->
-	<xacro:property name="Rwing" value="0.12"/>
+	<xacro:property name="Rwing" value="0.012"/>
 	<!-- mean chord length -->
-	<xacro:property name="cbar" value="0.06"/>
+	<xacro:property name="cbar" value="0.005"/>
 	<!-- vertical offset of wing attachment point from COM -->
-	<xacro:property name="d" value="0.1"/>
+	<xacro:property name="d" value="0.006"/>
 	<!-- Define materials -->
 	<material name="Black1">

Commit message: fix sign for hinge (now same for both wings)

File: urdf/sdab.xacro (robot description, xacro)
@@ -69,5 +69,5 @@
 			<parent link="${prefix}wing_spar"/>
 			<child link="${prefix}wing_membrane"/>
-			<axis xyz="0 ${-1 * sign} 0"/>
+			<axis xyz="0 -1 0"/>
 			<origin xyz="0.0 0 0.0" rpy="0 0 0"/>
 		</joint>

Commit message: body inertial params updated

File: urdf/sdab.xacro (robot description, xacro)
@@ -1,5 +1,5 @@
 <?xml version="1.0"?>
 <!--
-Units: mm, mg
+Units: m, kg
 Author: Avik De
 -->
@@ -19,4 +19,7 @@
 	<!-- vertical offset of wing attachment point from COM -->
 	<xacro:property name="d" value="0.006"/>
+	<!-- inertial properties -->
+	<xacro:property name="mb" value="0.055"/>
+	<xacro:property name="mwing" value="0.001"/>
 	<!-- Define materials -->
 	<material name="Black1">
@@ -36,6 +39,10 @@
 				<box size="${wbody} ${wbody} ${lbody}"/>
 			</geometry>
-	    <material name="Blue1"/>
-	   </visual>
+			<material name="Blue1"/>
+		 </visual>
+		<inertial>
+			<mass value="${mb}"/>
+			<inertia ixx="${1.0/12.0 * mb * (lbody*lbody + wbody*wbody)}" ixy="0.0" ixz="0.0" iyy="${1.0/12.0 * mb * (lbody*lbody + wbody*wbody)}" iyz="0.0" izz="${1.0/12.0 * mb * (wbody*wbody + wbody*wbody)}"/>
+		</inertial>
 	</link>
 	<!-- Define our wing macro -->
@@ -49,4 +56,8 @@
 				<material name="Black1"/>
 			</visual>
+		<inertial>
+			<mass value="${mwing}"/>
+			<inertia ixx="${1.0/12.0 * mb * (lbody*lbody + wbody*wbody)}" ixy="0.0" ixz="0.0" iyy="${1.0/12.0 * mb * (lbody*lbody + wbody*wbody)}" iyz="0.0" izz="${1.0/12.0 * mb * (wbody*wbody + wbody*wbody)}"/>
+		</inertial>
 		</link>
 		<link name="${prefix}wing_membrane">

Commit message: all known dynamic parameters added

File: urdf/sdab.xacro (robot description, xacro)
@@ -21,5 +21,11 @@
 	<!-- inertial properties -->
 	<xacro:property name="mb" value="0.055"/>
+	<xacro:property name="mspar" value="0.001"/>
 	<xacro:property name="mwing" value="0.001"/>
+	<!-- Stiffness and damping properties -->
+	<xacro:property name="dampingHinge" value="5e-10"/>
+	<xacro:property name="dampingSpar" value="0"/>
+	<xacro:property name="stiffnessHinge" value="1e-6"/>
+	<xacro:property name="stiffnessSpar" value="1e-6"/>
 	<!-- Define materials -->
 	<material name="Black1">
@@ -57,6 +63,6 @@
 			</visual>
 		<inertial>
-			<mass value="${mwing}"/>
-			<inertia ixx="${1.0/12.0 * mb * (lbody*lbody + wbody*wbody)}" ixy="0.0" ixz="0.0" iyy="${1.0/12.0 * mb * (lbody*lbody + wbody*wbody)}" iyz="0.0" izz="${1.0/12.0 * mb * (wbody*wbody + wbody*wbody)}"/>
+			<mass value="${mspar}"/>
+			<inertia ixx="${1.0/12.0 * mspar * ((Rwing+RwingOffset)*(Rwing+RwingOffset) + dspar*dspar)}" ixy="0.0" ixz="0.0" iyy="${1.0/12.0 * mspar * (2 * (Rwing+RwingOffset)*(Rwing+RwingOffset))}" iyz="0.0" izz="${1.0/12.0 * mspar * ((Rwing+RwingOffset)*(Rwing+RwingOffset) + dspar*dspar)}"/>
 		</inertial>
 		</link>
@@ -69,4 +75,8 @@
 				<material name="Gray1"/>
 			</visual>
+		<inertial>
+			<mass value="${mwing}"/>
+			<inertia ixx="${1.0/12.0 * mwing * (Rwing*Rwing + cbar*cbar)}" ixy="0.0" ixz="0.0" iyy="${1.0/12.0 * mwing * (dspar*dspar + cbar*cbar)}" iyz="0.0" izz="${1.0/12.0 * mwing * (dspar*dspar + Rwing*Rwing)}"/>
+		</inertial>
 		</link>
 		<!-- * * * Joint Definitions * * * -->
@@ -76,4 +86,5 @@
 			<axis xyz="0 0 ${-1 * sign}"/>
 			<origin xyz="0.0 0 ${d}" rpy="0 0 0"/>
+			<dynamics damping="${dampingSpar}" friction="0.0" spring_stiffness="${stiffnessSpar}" spring_reference="0"/>
 		</joint>
 		<joint name="${prefix}wing_hinge" type="continuous">
@@ -82,4 +93,5 @@
 			<axis xyz="0 -1 0"/>
 			<origin xyz="0.0 0 0.0" rpy="0 0 0"/>
+			<dynamics damping="${dampingHinge}" friction="0.0" spring_stiffness="${stiffnessHinge}" spring_reference="0"/>
 		</joint>
 	</xacro:macro>

Commit message: all dynamic parameters added to urdf including stiffnesses

File: urdf/sdab.xacro (robot description, xacro)
@@ -66,4 +66,9 @@
 			<inertia ixx="${1.0/12.0 * mspar * ((Rwing+RwingOffset)*(Rwing+RwingOffset) + dspar*dspar)}" ixy="0.0" ixz="0.0" iyy="${1.0/12.0 * mspar * (2 * (Rwing+RwingOffset)*(Rwing+RwingOffset))}" iyz="0.0" izz="${1.0/12.0 * mspar * ((Rwing+RwingOffset)*(Rwing+RwingOffset) + dspar*dspar)}"/>
 		</inertial>
+		<!-- pybullet does not expose spring_stiffness but does expose these so add them here too. We are not expecting contact -->
+		<contact>
+			<stiffness value="${stiffnessSpar}"/>
+			<damping value="${dampingSpar}"/>
+		</contact>
 		</link>
 		<link name="${prefix}wing_membrane">
@@ -79,4 +84,9 @@
 			<inertia ixx="${1.0/12.0 * mwing * (Rwing*Rwing + cbar*cbar)}" ixy="0.0" ixz="0.0" iyy="${1.0/12.0 * mwing * (dspar*dspar + cbar*cbar)}" iyz="0.0" izz="${1.0/12.0 * mwing * (dspar*dspar + Rwing*Rwing)}"/>
 		</inertial>
+		<!-- pybullet does not expose spring_stiffness but does expose these so add them here too. We are not expecting contact -->
+		<contact>
+			<stiffness value="${stiffnessHinge}"/>
+			<damping value="${dampingHinge}"/>
+		</contact>
 		</link>
 		<!-- * * * Joint Definitions * * * -->
@@ -91,5 +101,5 @@
 			<parent link="${prefix}wing_spar"/>
 			<child link="${prefix}wing_membrane"/>
-			<axis xyz="0 -1 0"/>
+			<axis xyz="0 1 0"/>
 			<origin xyz="0.0 0 0.0" rpy="0 0 0"/>
 			<dynamics damping="${dampingHinge}" friction="0.0" spring_stiffness="${stiffnessHinge}" spring_reference="0"/>

Commit message: make right spar red to identify

File: urdf/sdab.xacro (robot description, xacro)
@@ -32,4 +32,7 @@
 		<color rgba="0 0 0 1.0"/>
 	</material>
+	<material name="Red1">
+		<color rgba="1.0 0 0 1.0"/>
+	</material>
 	<material name="Gray1">
 		<color rgba="0 0 0 0.3"/>
@@ -53,5 +56,5 @@
 	</link>
 	<!-- Define our wing macro -->
-	<xacro:macro name="wing" params="sign prefix">
+	<xacro:macro name="wing" params="sign prefix sparcol">
 		<link name="${prefix}wing_spar">
 			<visual>
@@ -60,5 +63,5 @@
 					<box size="${dspar} ${RwingOffset + Rwing} ${dspar}"/>
 				</geometry>
-				<material name="Black1"/>
+				<material name="${sparcol}"/>
 			</visual>
 		<inertial>
@@ -107,5 +110,5 @@
 	</xacro:macro>
 	<!-- Two wings -->
-	<xacro:wing sign="-1" prefix="l" />
-	<xacro:wing sign="1" prefix="r" />
+	<xacro:wing sign="-1" prefix="l" sparcol="Black1"/>
+	<xacro:wing sign="1" prefix="r" sparcol="Red1"/>
 </robot>

Commit message: dynamics implemented as position control

File: urdf/sdab.xacro (robot description, xacro)
@@ -24,8 +24,8 @@
 	<xacro:property name="mwing" value="0.001"/>
 	<!-- Stiffness and damping properties -->
-	<xacro:property name="dampingHinge" value="5e-10"/>
+	<xacro:property name="stiffnessHinge" value="1e-2"/>
+	<xacro:property name="dampingHinge" value="1e-2"/>
+	<xacro:property name="stiffnessSpar" value="1e-6"/>
 	<xacro:property name="dampingSpar" value="0"/>
-	<xacro:property name="stiffnessHinge" value="1e-6"/>
-	<xacro:property name="stiffnessSpar" value="1e-6"/>
 	<!-- Define materials -->
 	<material name="Black1">
@@ -99,5 +99,5 @@
 			<axis xyz="0 0 ${-1 * sign}"/>
 			<origin xyz="0.0 0 ${d}" rpy="0 0 0"/>
-			<dynamics damping="${dampingSpar}" friction="0.0" spring_stiffness="${stiffnessSpar}" spring_reference="0"/>
+			<!-- <dynamics damping="${dampingSpar}" friction="0.0" spring_stiffness="${stiffnessSpar}" spring_reference="0"/> -->
 		</joint>
 		<joint name="${prefix}wing_hinge" type="continuous">
@@ -106,5 +106,5 @@
 			<axis xyz="0 1 0"/>
 			<origin xyz="0.0 0 0.0" rpy="0 0 0"/>
-			<dynamics damping="${dampingHinge}" friction="0.0" spring_stiffness="${stiffnessHinge}" spring_reference="0"/>
+			<!-- <dynamics damping="${dampingHinge}" friction="0.0" spring_stiffness="${stiffnessHinge}" spring_reference="0"/> -->
 		</joint>
 	</xacro:macro>

Commit message: limit is actually with the input frequency... need to tune flapping again

File: urdf/sdab.xacro (robot description, xacro)
@@ -24,6 +24,6 @@
 	<xacro:property name="mwing" value="0.001"/>
 	<!-- Stiffness and damping properties -->
-	<xacro:property name="stiffnessHinge" value="1e-2"/>
-	<xacro:property name="dampingHinge" value="1e-2"/>
+	<xacro:property name="stiffnessHinge" value="1e-8"/>
+	<xacro:property name="dampingHinge" value="1e-10"/>
 	<xacro:property name="stiffnessSpar" value="1e-6"/>
 	<xacro:property name="dampingSpar" value="0"/>

Commit message: fast frequency finally works

File: urdf/sdab.xacro (robot description, xacro)
@@ -24,6 +24,6 @@
 	<xacro:property name="mwing" value="0.001"/>
 	<!-- Stiffness and damping properties -->
-	<xacro:property name="stiffnessHinge" value="1e-8"/>
-	<xacro:property name="dampingHinge" value="1e-10"/>
+	<xacro:property name="stiffnessHinge" value="1e-4"/>
+	<xacro:property name="dampingHinge" value="1e-1"/>
 	<xacro:property name="stiffnessSpar" value="1e-6"/>
 	<xacro:property name="dampingSpar" value="0"/>

Commit message: nice flapping kinematics

File: urdf/sdab.xacro (robot description, xacro)
@@ -24,6 +24,6 @@
 	<xacro:property name="mwing" value="0.001"/>
 	<!-- Stiffness and damping properties -->
-	<xacro:property name="stiffnessHinge" value="1e-4"/>
-	<xacro:property name="dampingHinge" value="1e-1"/>
+	<xacro:property name="stiffnessHinge" value="1e-2"/>
+	<xacro:property name="dampingHinge" value="5e-3"/>
 	<xacro:property name="stiffnessSpar" value="1e-6"/>
 	<xacro:property name="dampingSpar" value="0"/>

Commit message: fix mass units

File: urdf/sdab.xacro (robot description, xacro)
@@ -20,10 +20,10 @@
 	<xacro:property name="d" value="0.006"/>
 	<!-- inertial properties -->
-	<xacro:property name="mb" value="0.055"/>
-	<xacro:property name="mspar" value="0.001"/>
-	<xacro:property name="mwing" value="0.001"/>
+	<xacro:property name="mb" value="55e-6"/>
+	<xacro:property name="mspar" value="1e-6"/>
+	<xacro:property name="mwing" value="1e-6"/>
 	<!-- Stiffness and damping properties -->
-	<xacro:property name="stiffnessHinge" value="1e-2"/>
-	<xacro:property name="dampingHinge" value="5e-3"/>
+	<xacro:property name="stiffnessHinge" value="5e-3"/>
+	<xacro:property name="dampingHinge" value="1e-3"/>
 	<xacro:property name="stiffnessSpar" value="1e-6"/>
 	<xacro:property name="dampingSpar" value="0"/>

Commit message: new flapping kinematics after mass fixed

File: urdf/sdab.xacro (robot description, xacro)
@@ -24,6 +24,6 @@
 	<xacro:property name="mwing" value="1e-6"/>
 	<!-- Stiffness and damping properties -->
-	<xacro:property name="stiffnessHinge" value="5e-3"/>
-	<xacro:property name="dampingHinge" value="1e-3"/>
+	<xacro:property name="stiffnessHinge" value="4e-1"/>
+	<xacro:property name="dampingHinge" value="4e-1"/>
 	<xacro:property name="stiffnessSpar" value="1e-6"/>
 	<xacro:property name="dampingSpar" value="0"/>

Commit message: can fly up with fake increased inertia

File: urdf/sdab.xacro (robot description, xacro)
@@ -24,6 +24,6 @@
 	<xacro:property name="mwing" value="1e-6"/>
 	<!-- Stiffness and damping properties -->
-	<xacro:property name="stiffnessHinge" value="4e-1"/>
-	<xacro:property name="dampingHinge" value="4e-1"/>
+	<xacro:property name="stiffnessHinge" value="2e-1"/>
+	<xacro:property name="dampingHinge" value="8e-1"/>
 	<xacro:property name="stiffnessSpar" value="1e-6"/>
 	<xacro:property name="dampingSpar" value="0"/>
@@ -52,5 +52,5 @@
 		<inertial>
 			<mass value="${mb}"/>
-			<inertia ixx="${1.0/12.0 * mb * (lbody*lbody + wbody*wbody)}" ixy="0.0" ixz="0.0" iyy="${1.0/12.0 * mb * (lbody*lbody + wbody*wbody)}" iyz="0.0" izz="${1.0/12.0 * mb * (wbody*wbody + wbody*wbody)}"/>
+			<inertia ixx="${10.0*1.0/12.0 * mb * (lbody*lbody + wbody*wbody)}" ixy="0.0" ixz="0.0" iyy="${10.0*1.0/12.0 * mb * (lbody*lbody + wbody*wbody)}" iyz="0.0" izz="${10.0*1.0/12.0 * mb * (wbody*wbody + wbody*wbody)}"/>
 		</inertial>
 	</link>

Commit message: flying

File: urdf/sdab.xacro (robot description, xacro)
@@ -20,10 +20,10 @@
 	<xacro:property name="d" value="0.006"/>
 	<!-- inertial properties -->
-	<xacro:property name="mb" value="55e-6"/>
+	<xacro:property name="mb" value="80e-6"/>
 	<xacro:property name="mspar" value="1e-6"/>
 	<xacro:property name="mwing" value="1e-6"/>
 	<!-- Stiffness and damping properties -->
-	<xacro:property name="stiffnessHinge" value="2e-1"/>
-	<xacro:property name="dampingHinge" value="8e-1"/>
+	<xacro:property name="stiffnessHinge" value="5e-1"/>
+	<xacro:property name="dampingHinge" value="5e-1"/>
 	<xacro:property name="stiffnessSpar" value="1e-6"/>
 	<xacro:property name="dampingSpar" value="0"/>

Commit message: flapping with force control but sensitive to params

File: urdf/sdab.xacro (robot description, xacro)
@@ -26,6 +26,6 @@
 	<xacro:property name="stiffnessHinge" value="5e-1"/>
 	<xacro:property name="dampingHinge" value="5e-1"/>
-	<xacro:property name="stiffnessSpar" value="1e-6"/>
-	<xacro:property name="dampingSpar" value="0"/>
+	<xacro:property name="stiffnessSpar" value="4e-5"/>
+	<xacro:property name="dampingSpar" value="7e-8"/>
 	<!-- Define materials -->
 	<material name="Black1">

Commit message: moving the fixme around

File: urdf/sdab.xacro (robot description, xacro)
@@ -24,6 +24,6 @@
 	<xacro:property name="mwing" value="1e-6"/>
 	<!-- Stiffness and damping properties -->
-	<xacro:property name="stiffnessHinge" value="5e-1"/>
-	<xacro:property name="dampingHinge" value="5e-1"/>
+	<xacro:property name="stiffnessHinge" value="2e-2"/>
+	<xacro:property name="dampingHinge" value="1e-2"/>
 	<xacro:property name="stiffnessSpar" value="4e-5"/>
 	<xacro:property name="dampingSpar" value="7e-8"/>

Commit message: seems to depend on d (which affects vertical position of COP)

File: urdf/sdab.xacro (robot description, xacro)
@@ -18,5 +18,5 @@
 	<xacro:property name="cbar" value="0.005"/>
 	<!-- vertical offset of wing attachment point from COM -->
-	<xacro:property name="d" value="0.006"/>
+	<xacro:property name="d" value="0.002"/>
 	<!-- inertial properties -->
 	<xacro:property name="mb" value="80e-6"/>

Commit message: change to mm mg ms

File: urdf/sdab.xacro (robot description, xacro)
@@ -7,25 +7,23 @@
 	<!-- Define parameters -->
 	<xacro:property name="pi" value="3.14159265359"/>
-	<xacro:property name="wbody" value="0.003"/>
-	<xacro:property name="lbody" value="0.012"/>
+	<xacro:property name="wbody" value="3"/>
+	<xacro:property name="lbody" value="12"/>
 	<!-- radial distance from center to start of wing -->
-	<xacro:property name="RwingOffset" value="0.004"/>
+	<xacro:property name="RwingOffset" value="4"/>
 	<!-- diameter of spar -->
-	<xacro:property name="dspar" value="0.001"/>
+	<xacro:property name="dspar" value="1"/>
 	<!-- radial wing length -->
-	<xacro:property name="Rwing" value="0.012"/>
+	<xacro:property name="Rwing" value="12"/>
 	<!-- mean chord length -->
-	<xacro:property name="cbar" value="0.005"/>
+	<xacro:property name="cbar" value="5"/>
 	<!-- vertical offset of wing attachment point from COM -->
-	<xacro:property name="d" value="0.002"/>
+	<xacro:property name="d" value="2"/>
 	<!-- inertial properties -->
-	<xacro:property name="mb" value="80e-6"/>
-	<xacro:property name="mspar" value="1e-6"/>
-	<xacro:property name="mwing" value="1e-6"/>
+	<xacro:property name="mb" value="80"/>
+	<xacro:property name="mspar" value="0.1"/>
+	<xacro:property name="mwing" value="0.55"/>
 	<!-- Stiffness and damping properties -->
-	<xacro:property name="stiffnessHinge" value="2e-2"/>
-	<xacro:property name="dampingHinge" value="1e-2"/>
-	<xacro:property name="stiffnessSpar" value="4e-5"/>
-	<xacro:property name="dampingSpar" value="7e-8"/>
+	<xacro:property name="whinge" value="2.5"/>
+	<xacro:property name="kstroke" value="65"/> <!-- total act = 240/T^2 + 30 -->
 	<!-- Define materials -->
 	<material name="Black1">
@@ -71,6 +69,6 @@
 		<!-- pybullet does not expose spring_stiffness but does expose these so add them here too. We are not expecting contact -->
 		<contact>
-			<stiffness value="${stiffnessSpar}"/>
-			<damping value="${dampingSpar}"/>
+			<stiffness value="${kstroke}"/>
+			<damping value="0"/>
 		</contact>
 		</link>
@@ -89,6 +87,6 @@
 		<!-- pybullet does not expose spring_stiffness but does expose these so add them here too. We are not expecting contact -->
 		<contact>
-			<stiffness value="${stiffnessHinge}"/>
-			<damping value="${dampingHinge}"/>
+			<stiffness value="${3*whinge}"/>
+			<damping value="${1.8*whinge}"/>
 		</contact>
 		</link>

Commit message: flappy wings no aero

File: urdf/sdab.xacro (robot description, xacro)
@@ -21,6 +21,6 @@
 	<!-- inertial properties -->
 	<xacro:property name="mb" value="80"/>
-	<xacro:property name="mspar" value="0.1"/>
-	<xacro:property name="mwing" value="0.55"/>
+	<xacro:property name="mspar" value="1"/>
+	<xacro:property name="mwing" value="1"/>
 	<!-- Stiffness and damping properties -->
 	<xacro:property name="whinge" value="2.5"/>

Commit message: update inertial properties; no mspar needed

File: urdf/sdab.xacro (robot description, xacro)
@@ -20,6 +20,8 @@
 	<xacro:property name="d" value="2"/>
 	<!-- inertial properties -->
-	<xacro:property name="mb" value="80"/>
-	<xacro:property name="mspar" value="1"/>
+	<xacro:property name="mb" value="100"/>
+	<xacro:property name="ixx" value="3333"/>
+	<xacro:property name="iyy" value="3333"/>
+	<xacro:property name="izz" value="1000"/>
 	<xacro:property name="mwing" value="1"/>
 	<!-- Stiffness and damping properties -->
@@ -50,5 +52,5 @@
 		<inertial>
 			<mass value="${mb}"/>
-			<inertia ixx="${10.0*1.0/12.0 * mb * (lbody*lbody + wbody*wbody)}" ixy="0.0" ixz="0.0" iyy="${10.0*1.0/12.0 * mb * (lbody*lbody + wbody*wbody)}" iyz="0.0" izz="${10.0*1.0/12.0 * mb * (wbody*wbody + wbody*wbody)}"/>
+			<inertia ixx="${ixx}" ixy="0.0" ixz="0.0" iyy="${iyy}" iyz="0.0" izz="${izz}"/>
 		</inertial>
 	</link>
@@ -64,6 +66,6 @@
 			</visual>
 		<inertial>
-			<mass value="${mspar}"/>
-			<inertia ixx="${1.0/12.0 * mspar * ((Rwing+RwingOffset)*(Rwing+RwingOffset) + dspar*dspar)}" ixy="0.0" ixz="0.0" iyy="${1.0/12.0 * mspar * (2 * (Rwing+RwingOffset)*(Rwing+RwingOffset))}" iyz="0.0" izz="${1.0/12.0 * mspar * ((Rwing+RwingOffset)*(Rwing+RwingOffset) + dspar*dspar)}"/>
+			<mass value="0"/>
+			<inertia ixx="0" ixy="0.0" ixz="0.0" iyy="0" iyz="0.0" izz="0"/>
 		</inertial>
 		<!-- pybullet does not expose spring_stiffness but does expose these so add them here too. We are not expecting contact -->

Commit message: force-controlled stroke works

File: urdf/sdab.xacro (robot description, xacro)
@@ -24,5 +24,5 @@
 	<xacro:property name="iyy" value="3333"/>
 	<xacro:property name="izz" value="1000"/>
-	<xacro:property name="mwing" value="1"/>
+	<xacro:property name="mwing" value="0.55"/>
 	<!-- Stiffness and damping properties -->
 	<xacro:property name="whinge" value="2.5"/>
