Commit message: URDF inertias tuned; should match the robot

File: urdf/sdab.xacro (robot description, xacro)
@@ -9,14 +9,6 @@
 	<xacro:property name="wbody" value="3"/>
 	<xacro:property name="lbody" value="12"/>
-	<!-- radial distance from center to start of wing -->
-	<xacro:property name="RwingOffset" value="4"/>
-	<!-- diameter of spar -->
-	<xacro:property name="dspar" value="1"/>
-	<!-- radial wing length -->
-	<xacro:property name="Rwing" value="12"/>
-	<!-- mean chord length -->
-	<xacro:property name="cbar" value="5"/>
 	<!-- vertical offset of wing attachment point from COM -->
-	<xacro:property name="d" value="2"/>
+	<xacro:property name="d" value="4"/>
 	<!-- inertial properties -->
 	<xacro:property name="mb" value="100"/>
@@ -24,5 +16,20 @@
 	<xacro:property name="iyy" value="3333"/>
 	<xacro:property name="izz" value="1000"/>
-	<xacro:property name="mwing" value="0.55"/>
+	<!-- See the mathematica file for how these were tuned to approximately match Jafferis (2016) -->
+	<xacro:property name="cbar" value="3.2"/>
+	<xacro:property name="dspar" value="0.5"/>
+	<!-- radial wing length *without the wing root offset*. Lw=Rwing+Rwingoffset -->
+	<!-- radial distance from center to start of wing -->
+	<xacro:property name="RwingOffset" value="3"/>
+	<xacro:property name="Rwing" value="14"/>
+	<xacro:property name="tmem" value="0.0015"/>
+	<xacro:property name="sparInertial">
+		<mass value="0.7"/>
+		<inertia ixx="0.0291667" ixy="0.0"  ixz="0.0" iyy="11.4479" iyz="0.0" izz="11.4479" />
+	</xacro:property>
+	<xacro:property name="memInertial">
+		<mass value="0.07"/>
+		<inertia ixx="0.0597333" ixy="0.0" ixz="0.0" iyy="1.20307" iyz="0.0" izz="1.14334" />
+	</xacro:property>
 	<!-- Stiffness and damping properties -->
 	<xacro:property name="whinge" value="2.5"/>
@@ -57,15 +64,15 @@
 	<!-- Define our wing macro -->
 	<xacro:macro name="wing" params="sign prefix sparcol">
+		<!--In robobee literature, "Ixx" = spanwise inertia, "Izz" = chordwise inertia. So, the wing frame has x along spar, z up, y pointing out of the wing plane. The first rpy below orients the frame so it is as expected.-->
 		<link name="${prefix}wing_spar">
 			<visual>
-				<origin xyz="0 ${sign * 0.5 * (Rwing + RwingOffset)} 0.0" rpy="0 0 0"/>
+				<origin xyz="0 ${sign*(0.5*Rwing)} 0.0" rpy="0 0 ${sign*0.5*pi}"/>
 				<geometry>
-					<box size="${dspar} ${RwingOffset + Rwing} ${dspar}"/>
+					<box size="${Rwing} ${dspar} ${dspar}"/>
 				</geometry>
 				<material name="${sparcol}"/>
 			</visual>
 		<inertial>
-			<mass value="0"/>
-			<inertia ixx="0" ixy="0.0" ixz="0.0" iyy="0" iyz="0.0" izz="0"/>
+			<xacro:insert_block name="sparInertial" />
 		</inertial>
 		<!-- pybullet does not expose spring_stiffness but does expose these so add them here too. We are not expecting contact -->
@@ -77,13 +84,12 @@
 		<link name="${prefix}wing_membrane">
 			<visual>
-				<origin xyz="0 ${sign * 0.5 * (Rwing + RwingOffset)} ${-0.5 * cbar}" rpy="0 0 0"/>
+				<origin xyz="0 ${sign*(0.5*Rwing)} ${-0.5 * cbar}" rpy="0 0 ${sign*0.5*pi}"/>
 				<geometry>
-					<box size="${dspar} ${Rwing} ${cbar}"/>
+					<box size="${Rwing} ${tmem} ${cbar}"/>
 				</geometry>
 				<material name="Gray1"/>
 			</visual>
 		<inertial>
-			<mass value="${mwing}"/>
-			<inertia ixx="${1.0/12.0 * mwing * (Rwing*Rwing + cbar*cbar)}" ixy="0.0" ixz="0.0" iyy="${1.0/12.0 * mwing * (dspar*dspar + cbar*cbar)}" iyz="0.0" izz="${1.0/12.0 * mwing * (dspar*dspar + Rwing*Rwing)}"/>
+			<xacro:insert_block name="memInertial" />
 		</inertial>
 		<!-- pybullet does not expose spring_stiffness but does expose these so add them here too. We are not expecting contact -->
@@ -98,5 +104,5 @@
 			<child link="${prefix}wing_spar"/>
 			<axis xyz="0 0 ${-1 * sign}"/>
-			<origin xyz="0.0 0 ${d}" rpy="0 0 0"/>
+			<origin xyz="0.0 ${sign*RwingOffset} ${d}" rpy="0 0 0"/>
 			<!-- <dynamics damping="${dampingSpar}" friction="0.0" spring_stiffness="${stiffnessSpar}" spring_reference="0"/> -->
 		</joint>

Commit message: trying to tune with sliders

File: urdf/sdab.xacro (robot description, xacro)
@@ -17,5 +17,5 @@
 	<xacro:property name="izz" value="1000"/>
 	<!-- See the mathematica file for how these were tuned to approximately match Jafferis (2016) -->
-	<xacro:property name="cbar" value="3.2"/>
+	<xacro:property name="cbar" value="4"/>
 	<xacro:property name="dspar" value="0.5"/>
 	<!-- radial wing length *without the wing root offset*. Lw=Rwing+Rwingoffset -->
@@ -25,13 +25,14 @@
 	<xacro:property name="tmem" value="0.0015"/>
 	<xacro:property name="sparInertial">
-		<mass value="0.7"/>
-		<inertia ixx="0.0291667" ixy="0.0"  ixz="0.0" iyy="11.4479" iyz="0.0" izz="11.4479" />
+		<mass value="0.72"/>
+		<inertia ixx="0.03" ixy="0" ixz="0" iyy="11.775" iyz="0" izz="11.775" />
 	</xacro:property>
 	<xacro:property name="memInertial">
-		<mass value="0.07"/>
-		<inertia ixx="0.0597333" ixy="0.0" ixz="0.0" iyy="1.20307" iyz="0.0" izz="1.14334" />
+		<mass value="0.06"/>
+		<inertia ixx="0.08" ixy="0.0" ixz="0.0" iyy="1.06" iyz="0.0" izz="0.981" />
 	</xacro:property>
 	<!-- Stiffness and damping properties -->
-	<xacro:property name="whinge" value="2.5"/>
+	<xacro:property name="khinge" value="3"/>
+	<xacro:property name="bhinge" value="2"/>
 	<xacro:property name="kstroke" value="65"/> <!-- total act = 240/T^2 + 30 -->
 	<!-- Define materials -->
@@ -95,6 +96,6 @@
 		<!-- pybullet does not expose spring_stiffness but does expose these so add them here too. We are not expecting contact -->
 		<contact>
-			<stiffness value="${3*whinge}"/>
-			<damping value="${1.8*whinge}"/>
+			<stiffness value="${khinge}"/>
+			<damping value="${bhinge}"/>
 		</contact>
 		</link>

Commit message: debugging applyExternalForce. kinematics fixed for left wing

File: urdf/sdab.xacro (robot description, xacro)
@@ -104,5 +104,5 @@
 			<parent link="body"/>
 			<child link="${prefix}wing_spar"/>
-			<axis xyz="0 0 ${-1 * sign}"/>
+			<axis xyz="0 0 ${sign}"/>
 			<origin xyz="0.0 ${sign*RwingOffset} ${d}" rpy="0 0 0"/>
 			<!-- <dynamics damping="${dampingSpar}" friction="0.0" spring_stiffness="${stiffnessSpar}" spring_reference="0"/> -->
@@ -111,5 +111,5 @@
 			<parent link="${prefix}wing_spar"/>
 			<child link="${prefix}wing_membrane"/>
-			<axis xyz="0 1 0"/>
+			<axis xyz="0 ${sign} 0"/>
 			<origin xyz="0.0 0 0.0" rpy="0 0 0"/>
 			<!-- <dynamics damping="${dampingHinge}" friction="0.0" spring_stiffness="${stiffnessHinge}" spring_reference="0"/> -->
@@ -117,5 +117,5 @@
 	</xacro:macro>
 	<!-- Two wings -->
-	<xacro:wing sign="-1" prefix="l" sparcol="Black1"/>
-	<xacro:wing sign="1" prefix="r" sparcol="Red1"/>
+	<xacro:wing sign="1" prefix="l" sparcol="Black1"/>
+	<xacro:wing sign="-1" prefix="r" sparcol="Red1"/>
 </robot>

Commit message: open-loop inputs work

File: urdf/sdab.xacro (robot description, xacro)
@@ -34,5 +34,5 @@
 	<!-- Stiffness and damping properties -->
 	<xacro:property name="khinge" value="3"/>
-	<xacro:property name="bhinge" value="2"/>
+	<xacro:property name="bhinge" value="4"/>
 	<xacro:property name="kstroke" value="65"/> <!-- total act = 240/T^2 + 30 -->
 	<!-- Define materials -->

Commit message: finally the external force makes sense

File: urdf/sdab.xacro (robot description, xacro)
@@ -34,5 +34,5 @@
 	<!-- Stiffness and damping properties -->
 	<xacro:property name="khinge" value="3"/>
-	<xacro:property name="bhinge" value="4"/>
+	<xacro:property name="bhinge" value="2"/>
 	<xacro:property name="kstroke" value="65"/> <!-- total act = 240/T^2 + 30 -->
 	<!-- Define materials -->
@@ -75,4 +75,5 @@
 			</visual>
 		<inertial>
+			<origin xyz="0 ${sign*(0.5*Rwing)} 0.0" rpy="0 0 ${sign*0.5*pi}"/>
 			<xacro:insert_block name="sparInertial" />
 		</inertial>
@@ -92,4 +93,5 @@
 			</visual>
 		<inertial>
+			<origin xyz="0 ${sign*(0.5*Rwing)} ${-0.5 * cbar}" rpy="0 0 ${sign*0.5*pi}"/>
 			<xacro:insert_block name="memInertial" />
 		</inertial>

Commit message: SDAB model make 3D pybullet sim usable (#158)
* rename to model

* change to mm mg ms

* flappy wings no aero

* smaller timestep

* flaps and rises, but hinge dynamics don't make sense, and gravity cannot be enabled yet

* major reorg

* another large reorg

* update inertial properties; no mspar needed

* force-controlled stroke works

* manual hinge PD control seems to have the same result as PD_CONTROL using pybullet. doesn't work

* call xacro from here

* clean up a bit

* tune wing inertias for URDF

* URDF inertias tuned; should match the robot

* trying to tune with sliders

* at least confirmed that applyExternalForce is doing something

* debugging applyExternalForce. kinematics fixed for left wing

* pcop is correct

* now the deflection looks OK for the force with a lot of transformations

* now flaps

* actual hinge dynamics works!!

* open-loop inputs work

* easy-to-access testF mode

* this one doesn't work either and is the same

* the deflection is correct when rcopnondim>1. at =1 it does nothing

* create a test urdf

* example works

* fixed - update to pybullet 2.8.2

* finally the external force makes sense

* need pybullet 2.8.2

* working full openloop control

* can add back gravity

File: urdf/sdab.xacro (robot description, xacro)
@@ -7,25 +7,33 @@
 	<!-- Define parameters -->
 	<xacro:property name="pi" value="3.14159265359"/>
-	<xacro:property name="wbody" value="0.003"/>
-	<xacro:property name="lbody" value="0.012"/>
+	<xacro:property name="wbody" value="3"/>
+	<xacro:property name="lbody" value="12"/>
+	<!-- vertical offset of wing attachment point from COM -->
+	<xacro:property name="d" value="4"/>
+	<!-- inertial properties -->
+	<xacro:property name="mb" value="100"/>
+	<xacro:property name="ixx" value="3333"/>
+	<xacro:property name="iyy" value="3333"/>
+	<xacro:property name="izz" value="1000"/>
+	<!-- See the mathematica file for how these were tuned to approximately match Jafferis (2016) -->
+	<xacro:property name="cbar" value="4"/>
+	<xacro:property name="dspar" value="0.5"/>
+	<!-- radial wing length *without the wing root offset*. Lw=Rwing+Rwingoffset -->
 	<!-- radial distance from center to start of wing -->
-	<xacro:property name="RwingOffset" value="0.004"/>
-	<!-- diameter of spar -->
-	<xacro:property name="dspar" value="0.001"/>
-	<!-- radial wing length -->
-	<xacro:property name="Rwing" value="0.012"/>
-	<!-- mean chord length -->
-	<xacro:property name="cbar" value="0.005"/>
-	<!-- vertical offset of wing attachment point from COM -->
-	<xacro:property name="d" value="0.002"/>
-	<!-- inertial properties -->
-	<xacro:property name="mb" value="80e-6"/>
-	<xacro:property name="mspar" value="1e-6"/>
-	<xacro:property name="mwing" value="1e-6"/>
+	<xacro:property name="RwingOffset" value="3"/>
+	<xacro:property name="Rwing" value="14"/>
+	<xacro:property name="tmem" value="0.0015"/>
+	<xacro:property name="sparInertial">
+		<mass value="0.72"/>
+		<inertia ixx="0.03" ixy="0" ixz="0" iyy="11.775" iyz="0" izz="11.775" />
+	</xacro:property>
+	<xacro:property name="memInertial">
+		<mass value="0.06"/>
+		<inertia ixx="0.08" ixy="0.0" ixz="0.0" iyy="1.06" iyz="0.0" izz="0.981" />
+	</xacro:property>
 	<!-- Stiffness and damping properties -->
-	<xacro:property name="stiffnessHinge" value="2e-2"/>
-	<xacro:property name="dampingHinge" value="1e-2"/>
-	<xacro:property name="stiffnessSpar" value="4e-5"/>
-	<xacro:property name="dampingSpar" value="7e-8"/>
+	<xacro:property name="khinge" value="3"/>
+	<xacro:property name="bhinge" value="2"/>
+	<xacro:property name="kstroke" value="65"/> <!-- total act = 240/T^2 + 30 -->
 	<!-- Define materials -->
 	<material name="Black1">
@@ -52,43 +60,44 @@
 		<inertial>
 			<mass value="${mb}"/>
-			<inertia ixx="${10.0*1.0/12.0 * mb * (lbody*lbody + wbody*wbody)}" ixy="0.0" ixz="0.0" iyy="${10.0*1.0/12.0 * mb * (lbody*lbody + wbody*wbody)}" iyz="0.0" izz="${10.0*1.0/12.0 * mb * (wbody*wbody + wbody*wbody)}"/>
+			<inertia ixx="${ixx}" ixy="0.0" ixz="0.0" iyy="${iyy}" iyz="0.0" izz="${izz}"/>
 		</inertial>
 	</link>
 	<!-- Define our wing macro -->
 	<xacro:macro name="wing" params="sign prefix sparcol">
+		<!--In robobee literature, "Ixx" = spanwise inertia, "Izz" = chordwise inertia. So, the wing frame has x along spar, z up, y pointing out of the wing plane. The first rpy below orients the frame so it is as expected.-->
 		<link name="${prefix}wing_spar">
 			<visual>
-				<origin xyz="0 ${sign * 0.5 * (Rwing + RwingOffset)} 0.0" rpy="0 0 0"/>
+				<origin xyz="0 ${sign*(0.5*Rwing)} 0.0" rpy="0 0 ${sign*0.5*pi}"/>
 				<geometry>
-					<box size="${dspar} ${RwingOffset + Rwing} ${dspar}"/>
+					<box size="${Rwing} ${dspar} ${dspar}"/>
 				</geometry>
 				<material name="${sparcol}"/>
 			</visual>
 		<inertial>
-			<mass value="${mspar}"/>
-			<inertia ixx="${1.0/12.0 * mspar * ((Rwing+RwingOffset)*(Rwing+RwingOffset) + dspar*dspar)}" ixy="0.0" ixz="0.0" iyy="${1.0/12.0 * mspar * (2 * (Rwing+RwingOffset)*(Rwing+RwingOffset))}" iyz="0.0" izz="${1.0/12.0 * mspar * ((Rwing+RwingOffset)*(Rwing+RwingOffset) + dspar*dspar)}"/>
+			<origin xyz="0 ${sign*(0.5*Rwing)} 0.0" rpy="0 0 ${sign*0.5*pi}"/>
+			<xacro:insert_block name="sparInertial" />
 		</inertial>
 		<!-- pybullet does not expose spring_stiffness but does expose these so add them here too. We are not expecting contact -->
 		<contact>
-			<stiffness value="${stiffnessSpar}"/>
-			<damping value="${dampingSpar}"/>
+			<stiffness value="${kstroke}"/>
+			<damping value="0"/>
 		</contact>
 		</link>
 		<link name="${prefix}wing_membrane">
 			<visual>
-				<origin xyz="0 ${sign * 0.5 * (Rwing + RwingOffset)} ${-0.5 * cbar}" rpy="0 0 0"/>
+				<origin xyz="0 ${sign*(0.5*Rwing)} ${-0.5 * cbar}" rpy="0 0 ${sign*0.5*pi}"/>
 				<geometry>
-					<box size="${dspar} ${Rwing} ${cbar}"/>
+					<box size="${Rwing} ${tmem} ${cbar}"/>
 				</geometry>
 				<material name="Gray1"/>
 			</visual>
 		<inertial>
-			<mass value="${mwing}"/>
-			<inertia ixx="${1.0/12.0 * mwing * (Rwing*Rwing + cbar*cbar)}" ixy="0.0" ixz="0.0" iyy="${1.0/12.0 * mwing * (dspar*dspar + cbar*cbar)}" iyz="0.0" izz="${1.0/12.0 * mwing * (dspar*dspar + Rwing*Rwing)}"/>
+			<origin xyz="0 ${sign*(0.5*Rwing)} ${-0.5 * cbar}" rpy="0 0 ${sign*0.5*pi}"/>
+			<xacro:insert_block name="memInertial" />
 		</inertial>
 		<!-- pybullet does not expose spring_stiffness but does expose these so add them here too. We are not expecting contact -->
 		<contact>
-			<stiffness value="${stiffnessHinge}"/>
-			<damping value="${dampingHinge}"/>
+			<stiffness value="${khinge}"/>
+			<damping value="${bhinge}"/>
 		</contact>
 		</link>
@@ -97,6 +106,6 @@
 			<parent link="body"/>
 			<child link="${prefix}wing_spar"/>
-			<axis xyz="0 0 ${-1 * sign}"/>
-			<origin xyz="0.0 0 ${d}" rpy="0 0 0"/>
+			<axis xyz="0 0 ${sign}"/>
+			<origin xyz="0.0 ${sign*RwingOffset} ${d}" rpy="0 0 0"/>
 			<!-- <dynamics damping="${dampingSpar}" friction="0.0" spring_stiffness="${stiffnessSpar}" spring_reference="0"/> -->
 		</joint>
@@ -104,5 +113,5 @@
 			<parent link="${prefix}wing_spar"/>
 			<child link="${prefix}wing_membrane"/>
-			<axis xyz="0 1 0"/>
+			<axis xyz="0 ${sign} 0"/>
 			<origin xyz="0.0 0 0.0" rpy="0 0 0"/>
 			<!-- <dynamics damping="${dampingHinge}" friction="0.0" spring_stiffness="${stiffnessHinge}" spring_reference="0"/> -->
@@ -110,5 +119,5 @@
 	</xacro:macro>
 	<!-- Two wings -->
-	<xacro:wing sign="-1" prefix="l" sparcol="Black1"/>
-	<xacro:wing sign="1" prefix="r" sparcol="Red1"/>
+	<xacro:wing sign="1" prefix="l" sparcol="Black1"/>
+	<xacro:wing sign="-1" prefix="r" sparcol="Red1"/>
 </robot>

Commit message: replaced aero model with the one in julia

File: urdf/sdab.xacro (robot description, xacro)
@@ -34,5 +34,5 @@
 	<!-- Stiffness and damping properties -->
 	<xacro:property name="khinge" value="3"/>
-	<xacro:property name="bhinge" value="2"/>
+	<xacro:property name="bhinge" value="3"/>
 	<xacro:property name="kstroke" value="65"/> <!-- total act = 240/T^2 + 30 -->
 	<!-- Define materials -->

Commit message: some tuning

File: urdf/sdab.xacro (robot description, xacro)
@@ -34,5 +34,5 @@
 	<!-- Stiffness and damping properties -->
 	<xacro:property name="khinge" value="3"/>
-	<xacro:property name="bhinge" value="3"/>
+	<xacro:property name="bhinge" value="2"/>
 	<xacro:property name="kstroke" value="65"/> <!-- total act = 240/T^2 + 30 -->
 	<!-- Define materials -->
