Commit message: example works

File: template/test2link.urdf (robot description, URDF)
Before this commit: robot test2link, 3 links, 2 joints
Links:
- link body: mass None -> 1
- link link1: mass None -> 1
- link link2: mass None -> 10
Joints:
- joint 1: origin xyz=0 1 -0.3 rpy=0 0 0 -> xyz=0 1 -0.1 rpy=0 0 0
